File: 5251/5251.kicad_pcb (KiCad board)
At the start: 2 copper layers, 424 x 139.2 mm, 92 parts, among them J1 Conn_01x30, U1 F1_SENSE, U10 5, U11 6, U12 7, U13 8, U14 9, U15 0, U16 -_, U17 =+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

Commit message: inprogress changes made with an alternate backplane
Routing:
- net GNDA: track 5695.2 -> 188.2 mm
